File: Supply_Power.kicad_pcb (KiCad board)
At the start: 2 copper layers, 105.9 x 49.3 mm, 35 parts, among them J1 +3.3V, J2 V_IN, J3 +15V, J4 +5V_CAN, J5 +5V, U1 R-785.0-1.0, U2 R-78C3.3-1.0

Commit message: Первая версия в производство
Parts:
- added J6: +5V, Connector_Molex:Molex_Micro-Fit_3.0_43045-0400_2x02_P3.00mm_Horizontal, F.Cu at (113.3, 34.6)
- added J7: +5V, Connector_Molex:Molex_Micro-Fit_3.0_43045-0400_2x02_P3.00mm_Horizontal, F.Cu at (124.7, 34.6)
- L1, L2: footprint Inductor_SMD:L_1210_3225Metric_Pad1.42x2.65mm_HandSolder -> Inductor_SMD:L_1812_4532Metric_Pad1.30x3.40mm_HandSolder
- moved H2 22.5 mm to (160.0, 27.4)
- moved J4 22.4 mm to (148.6, 34.6)
- moved J1 22.4 mm to (136.7, 34.6)
- moved H3 22.4 mm to (160.0, 69.1)
- moved H1 2.79 mm to (39.1, 27.4)
- moved H4 0.25 mm to (39.1, 69.1)
- moved L1 0.25 mm to (47.2, 44.5)
- moved L2 0.25 mm to (47.2, 58.2)
Routing:
- net +3V3: track 60.2 -> 82.8 mm
- net +5VD: track 74.0 -> 95.8 mm
Other:
- board size 105.9 x 49.3 mm -> 128.5 x 49.3 mm
