File: Supply_Power.kicad_sch (KiCad schematic)
At the start: 35 parts, among them J1 +3.3V, J2 V_IN, J3 +15V, J4 +5V_CAN, J5 +5V, U1 R-785.0-1.0, U2 R-78C3.3-1.0

Commit message: Первая версия в производство
Parts:
- added J6, J7: +5V, Connector_Molex:Molex_Micro-Fit_3.0_43045-0400_2x02_P3.00mm_Horizontal, symbol Connector_Generic:Conn_02x02_Odd_Even
- L1, L2: footprint Inductor_SMD:L_1210_3225Metric_Pad1.42x2.65mm_HandSolder -> Inductor_SMD:L_1812_4532Metric_Pad1.30x3.40mm_HandSolder
Connections:
- net +5V: now also J6.2 (Pin_2), J6.4 (Pin_4), J7.2 (Pin_2), J7.4 (Pin_4)
- net GND: now also J6.1 (Pin_1), J6.3 (Pin_3), J7.1 (Pin_1), J7.3 (Pin_3)
